File: hardware/Artembed.sch (EAGLE design)
At the start: 97 parts, among them J3 CORTEX_JTAG_DEBUG_PTH_NS, J4 CORTEX_JTAG_DEBUG_MINIMUM_PTH, J7 CAMERA-HIMAX, U1 ARTEMIS_MODULESMD, U2 LIS2DH12, U3 1.8V, Y1 16MHz, Y2 32.768kHz

Commit message: progress commit
got a lot of routing done, but more to do
Parts:
- removed C22, C23: 1.0uF, ambiq:1.0UF-0402-TIGHT-16V-10%
- removed R32: 10k, SparkFun-Resistors:10KOHM-0402T-1/16W-1%
- removed S1: MOMENTARY-SWITCH-SPST-SMD-5.2MM-TALL, SparkFun-Switches:MOMENTARY-SWITCH-SPST-SMD-5.2MM-TALL
- removed TP14, TP15, TP16, TP17, TP18, TP6, TP7, TP8: TEST-POINT3X5, SparkFun-Connectors:TEST-POINT3X5
- removed U$1: DAPLINK_KL26Z, artembed:DAPLINK_KL26Z
- removed Y2: 32.768kHz, SparkFun-Clocks:CRYSTAL-32.768KHZSMD-3.2X1.5
- added C18: 10uF, SparkFun-Capacitors:10UF-0603-6.3V-20%
- added C19: 1.0uF, SparkFun-Capacitors:1.0UF-0603-16V-10%
- added J9: (no value), SparkFun-Connectors:CONN_07NO_SILK
- added R30: 10k, SparkFun-Resistors:10KOHM-0603-1/10W-1%
- added S3: RESET IF, SparkFun-Switches:MOMENTARY-SWITCH-SPST-SMD-4.6X2.8MM
- added U4: 1.8V, SparkFun-IC-Power:V_REG_AP2127K-1.8V
- added U5: LIS2DH12, SparkFun-Sensors:LIS2DH12
- C10: value 10uF -> 8pF; device SparkFun-Capacitors:10UF-0603-6.3V-20% -> SparkFun-Capacitors:CAP-0603
- C11, C17: value 1.0uF -> 0.1uF; device SparkFun-Capacitors:1.0UF-0603-16V-10% -> SparkFun-Capacitors:0.1UF-0603-25V-5%
- C12, C3: value 0.1uF -> 1.0uF; device SparkFun-Capacitors:0.1UF-0603-25V-5% -> SparkFun-Capacitors:1.0UF-0603-16V-10%
- C13: value 15pF -> 0.1uF; device SparkFun-Capacitors:15PF-0603-50V-5% -> SparkFun-Capacitors:0.1UF-0603-25V-5%
- C15: value 1nF -> 15pF; device SparkFun-Capacitors:1.0NF/1000PF-0603-50V-10% -> SparkFun-Capacitors:15PF-0603-50V-5%
- C2: value 1.0uF -> 10uF; device SparkFun-Capacitors:1.0UF-0603-16V-10% -> SparkFun-Capacitors:10UF-0603-6.3V-20%
- C20: value 0.1uF -> 1.0uF; device ambiq:0.1UF-0402-TIGHT-16V-10% -> SparkFun-Capacitors:1.0UF-0603-16V-10%
- C21: value 10uF -> 1.0uF; device SparkFun-Capacitors:10UF-0603-6.3V-20% -> SparkFun-Capacitors:1.0UF-0603-16V-10%
- C5: value 2.2uF -> 1nF; device SparkFun-Capacitors:2.2UF-0603-10V-20% -> SparkFun-Capacitors:1.0NF/1000PF-0603-50V-10%
- C6: value 0.1uF -> 2.2uF; device SparkFun-Capacitors:0.1UF-0603-25V-5% -> SparkFun-Capacitors:2.2UF-0603-10V-20%
- C8: value 22pF -> 0.1uF; device SparkFun-Capacitors:22PF-0603-50V-5% -> SparkFun-Capacitors:0.1UF-0603-25V-5%
- C9: value 22pF -> 8pF; device SparkFun-Capacitors:22PF-0603-50V-5% -> SparkFun-Capacitors:CAP-0603
- D1: value RED -> 3A/10V/280mV; device SparkFun-LED:LED-RED0603 -> SparkFun-DiscreteSemi:DIODE-SCHOTTKY-BAT60A
- D2: value BLUE -> 3A/10V/280mV; device SparkFun-LED:LED-BLUE0603 -> SparkFun-DiscreteSemi:DIODE-SCHOTTKY-BAT60A
- D3: value GREEN -> PRTR5V0U2F; device SparkFun-LED:LED-GREEN0603 -> SparkFun-IC-Power:PRTR5V0U2F
- D4: value Yellow -> BLUE; device SparkFun-LED:LED-YELLOW0603 -> SparkFun-LED:LED-BLUE0603
- D5: value PRTR5V0U2F -> GREEN; device SparkFun-IC-Power:PRTR5V0U2F -> SparkFun-LED:LED-GREEN0603
- D6: value 3A/10V/280mV -> Yellow; device SparkFun-DiscreteSemi:DIODE-SCHOTTKY-BAT60A -> SparkFun-LED:LED-YELLOW0603
- D7: value 3A/10V/280mV -> RED; device SparkFun-DiscreteSemi:DIODE-SCHOTTKY-BAT60A -> SparkFun-LED:LED-RED0603
- J1: device SparkFun-Connectors:USB_C2-LAYER -> SparkFun-Connectors:CONN_02-JST-2MM-SMT
- J2: device SparkFun-Connectors:CONN_02-JST-2MM-SMT -> SparkFun-Connectors:USB_C2-LAYER
- J3: value CORTEX_JTAG_DEBUG_PTH_NS -> CORTEX_JTAG_DEBUG_MINIMUM_PTH; device SparkFun-Connectors:CORTEX_JTAG_DEBUG_PTH_NS -> SparkFun-Connectors:CORTEX_JTAG_DEBUG_MINIMUM_PTH
- J4: value CORTEX_JTAG_DEBUG_MINIMUM_PTH -> CORTEX_JTAG_DEBUG_PTH_NS; device SparkFun-Connectors:CORTEX_JTAG_DEBUG_MINIMUM_PTH -> SparkFun-Connectors:CORTEX_JTAG_DEBUG_PTH_NS
- J5: device SparkFun-Connectors:QWIIC_CONNECTORJS-1MM -> SparkFun-Connectors:CONN_08NO_SILK_FEMALE_PTH
- J6: device SparkFun-Connectors:CONN_08" -> SparkFun-Connectors:CONN_07NO_SILK
- J8: device SparkFun-Connectors:CONN_08" -> SparkFun-Connectors:QWIIC_CONNECTORJS-1MM
- R10: value 330 -> DNP; device SparkFun-Resistors:330OHM-0603-1/10W-1% -> SparkFun-Resistors:RESISTOR0603
- R11: value 10k -> DNP; device SparkFun-Resistors:10KOHM-0603-1/10W-1% -> SparkFun-Resistors:RESISTOR0603
- R12: value 5.62k -> 0; device SparkFun-Resistors:5.62KOHM-0603-1/10W-1% -> SparkFun-Resistors:0OHM-0603-1/10W
- R13: value 10k -> 0; device SparkFun-Resistors:10KOHM-0603-1/10W-1% -> SparkFun-Resistors:0OHM-0603-1/10W
- R14: value DNP -> 5.62k; device SparkFun-Resistors:RESISTOR0603 -> SparkFun-Resistors:5.62KOHM-0603-1/10W-1%
- R19: value DNP -> 10k; device SparkFun-Resistors:RESISTOR0603 -> SparkFun-Resistors:10KOHM-0603-1/10W-1%
- R2, R3: value 330 -> 10k; device SparkFun-Resistors:330OHM-0603-1/10W-1% -> SparkFun-Resistors:10KOHM-0603-1/10W-1%
- R20: value DNP -> 2.2k; device SparkFun-Resistors:RESISTOR0603 -> SparkFun-Resistors:2.2KOHM-0603-1/10W-1%
- R21: value 10k -> 2.2k; device SparkFun-Resistors:10KOHM-0603-1/10W-1% -> SparkFun-Resistors:2.2KOHM-0603-1/10W-1%
- R22: value 0 -> 10k; device SparkFun-Resistors:0OHM-0603-1/10W -> SparkFun-Resistors:10KOHM-0603-1/10W-1%
- R23: value 0 -> 33; device SparkFun-Resistors:0OHM-0603-1/10W -> SparkFun-Resistors:33OHM-0603-1/10W-1%
- R24: value 0 -> 10; device SparkFun-Resistors:0OHM-0603-1/10W -> SparkFun-Resistors:10OHM-0603-1/10W-1%
- R25, R26: value 0 -> 330; device SparkFun-Resistors:0OHM-0603-1/10W -> SparkFun-Resistors:330OHM-0603-1/10W-1%
- R27: value 10k -> 330; device SparkFun-Resistors:10KOHM-0603-1/10W-1% -> SparkFun-Resistors:330OHM-0603-1/10W-1%
- R28: value 2.2k -> 330; device SparkFun-Resistors:2.2KOHM-0603-1/10W-1% -> SparkFun-Resistors:330OHM-0603-1/10W-1%
- R29: value 2.2k -> 33; device SparkFun-Resistors:2.2KOHM-0603-1/10W-1% -> SparkFun-Resistors:33OHM-0603-1/10W-1%
- R4: value 330 -> 0; device SparkFun-Resistors:330OHM-0603-1/10W-1% -> SparkFun-Resistors:0OHM-0603-1/10W
- R5, R6: value 5.1k -> 0; device SparkFun-Resistors:5.1KOHM5.1KOHM-0603-1/10W-1% -> SparkFun-Resistors:0OHM-0603-1/10W
- R7, R8: value 33 -> 5.1k; device SparkFun-Resistors:33OHM-0603-1/10W-1% -> SparkFun-Resistors:5.1KOHM5.1KOHM-0603-1/10W-1%
- R9: value 10 -> 0; device SparkFun-Resistors:10OHM-0603-1/10W-1% -> SparkFun-Resistors:0OHM-0603-1/10W
- S2: value MOMENTARY-SWITCH-SPST-SMD-5.2MM-TALL -> RESET TGT; device SparkFun-Switches:MOMENTARY-SWITCH-SPST-SMD-5.2MM-TALL -> SparkFun-Switches:MOMENTARY-SWITCH-SPST-SMD-4.6X2.8MM
- U1: value ARTEMIS_MODULESMD -> DAPLINK_KL26Z; device SparkFun-IC-Microcontroller:ARTEMIS_MODULESMD -> artembed:DAPLINK_KL26Z
- U2: value LIS2DH12 -> 16MHz; device SparkFun-Sensors:LIS2DH12 -> SparkFun-Clocks:CRYSTAL-16MHZ_SMALL
- U3: value 1.8V -> ARTEMIS_MODULESMD; device SparkFun-IC-Power:V_REG_AP2127K-1.8V -> SparkFun-IC-Microcontroller:ARTEMIS_MODULESMD
- Y1: value 16MHz -> 32.768kHz; device SparkFun-Clocks:CRYSTAL-16MHZSMD-5X3.2 -> SparkFun-Clocks:CRYSTAL-32.768KHZSMD-3.2X1.5
Connections:
- removed net N$12: C6.1, C7.1, U$1.VDD, U$1.VDDA
- removed net N$6: D5.5, R9.1
- new net D10: J9.4, U3.(SLNCE/I2SWCLK)D3
- new net D11: J9.5, U3.(SLMISO)D2
- new net D12: J9.6, U3.(SLMOSI/SLSDA)D1
- new net D13: J9.7, U3.(SLSCK/SLSCL/CLKOUT)D0
- new net D7: J9.1, U3.~AD13(I2SBCLK/RX1)
- new net D8: J9.2, U3.~AD29(PDMDATA)
- new net D9: J9.3, U3.(RX1/SLINT)~D4
- net !RST: now also C11.1, J4.!RESET, R14.1, R19.2, U1.IF_NRESET, U1.USB_VBUS; no longer C4.1, J3.!RESET, R11.2, R12.1, TP7.1, U$1.IF_NRESET, U$1.USB_VBUS
- net !TGT_RST: now also R9.2, S3.2, TP11.1, U1.NRESET_FB_ISP; no longer J4.!RESET, R20.1, S1.2, TP1.1, U$1.NRESET_FB_ISP
- net !TGT_RST!_HW: now also C5.1, J3.!RESET, R3.1, U3.!RST; no longer C15.1, R21.1, U1.!RST
- net !TGT_RST!_SW: now also U3.(CMPRF0/SCCCLK/I2SBCLK)~D19; no longer U1.(CMPRF0/SCCCLK/I2SBCLK)~D19
- net 1.8V: now also C16.1, TP1.1, U4.OUT; no longer C23.1, TP18.1, U3.OUT
- net 3.3V: now also C6.1, C7.1, C8.1, D1.A, J4.VCC, R11.2, R25.2, R26.2, R27.2, R28.2, TP13.1, U1.VDD, U1.VDDA, U1.VOUT33; no longer C5.1, D7.A, J3.VCC, R13.2, R14.2, R19.2, R3.2, R4.2, TP11.1, U$1.VOUT33
- net CAMERA_D0: now also U3.(MOSI3/RX1)D38; no longer U1.(MOSI3/RX1)D38
- net CAMERA_D1: now also U3.(SCL4/SCK4/TX1)~D39; no longer U1.(SCL4/SCK4/TX1)~D39
- net CAMERA_D2: now also U3.(SDA4/MISO4/RX1)D40; no longer U1.(SDA4/MISO4/RX1)D40
- net CAMERA_D3: now also U3.(BLEIF_IRQ/SWO/I2SWCLK)D41; no longer U1.(BLEIF_IRQ/SWO/I2SWCLK)D41
- net CAMERA_D4: now also U3.(SCL3/SCK3/TX1)~D42; no longer U1.(SCL3/SCK3/TX1)~D42
- net CAMERA_D5: now also U3.(SDA3/MISO3/RX1)~D43; no longer U1.(SDA3/MISO3/RX1)~D43
- net CAMERA_D6: now also U3.(MOSI4)~D44; no longer U1.(MOSI4)~D44
- net CAMERA_D7: now also U3.(SWO/I2SDAT/PDMDATA)~D45; no longer U1.(SWO/I2SDAT/PDMDATA)~D45
- net CAMERA_DVDD_EN: now also R30.2, U3.(MOSI1/TX1/PDMCLK)D10, U4.EN; no longer R32.2, U1.(MOSI1/TX1/PDMCLK)D10, U3.EN
- net CAMERA_HSYNC: now also U3.(RX1/TRIG1/PDMDATA)D36; no longer U1.(RX1/TRIG1/PDMDATA)D36
- net CAMERA_INT: now also U3.(TX1/32KHZ/SWO)~D24; no longer U1.(TX1/32KHZ/SWO)~D24
- net CAMERA_MCLK: now also U3.(SCCRST)~D26; no longer U1.(SCCRST)~D26
- net CAMERA_PCLK: now also U3.(MOSI2/I2SWCLK)~D28; no longer U1.(MOSI2/I2SWCLK)~D28
- net CAMERA_TRIG: now also U3.(I2SWCLK/CMPOUT)~D23; no longer U1.(I2SWCLK/CMPOUT)~D23
- net CAMERA_VSYNC: now also U3.(TX1/PDMCLK/SCCIO)~D37; no longer U1.(TX1/PDMCLK/SCCIO)~D37
- net D1_SLSDA: now also J5.1; no longer J8.1
- net D2_SLSCL: now also J5.2; no longer J8.2
- net D3_PWM_UARTTX: now also J5.3, U3.~AD35(TX1/I2SDAT/PDMCLK); no longer J8.3, U1.~AD35(TX1/I2SDAT/PDMCLK)
- net D4_MISO: now also J5.4, U3.(SDA0/MISO0/I2SDAT)~D6; no longer J8.4, U1.(SDA0/MISO0/I2SDAT)~D6
- net D5_MOSI_CLKOUT: now also J5.5, U3.(MOSI0/CLKOUT)~D7; no longer J8.5, U1.(MOSI0/CLKOUT)~D7
- net D6_SCLK: now also J5.6, U3.(SCL0/SCK0)~D5; no longer J8.6, U1.(SCL0/SCK0)~D5
- net GND: now also C13.2, C15.1, C18.2, C19.2, D3.2, D7.C, J1.1, J2.GND, J3.GND, J4.GND@3, J4.GND@5, J4.GNDDTCT, J5.8, J8.1, R19.1, R22.1, R30.1, R7.1, R8.1, S3.1, TP9.1, U1.VSS1, U1.VSS2, U1.VSSA, U3.GND*6, U4.GND, U5.GND, U5.RES; no longer C13.1, C15.2, C22.2, C23.2, D1.C, D5.2, J1.GND, J2.1, J3.GND@3, J3.GND@5, J3.GNDDTCT, J4.GND, J5.1, J6.8, J8.8, R11.1, R27.1, R32.1, R5.1, R6.1, S1.1, TP8.1, U$1.VSS1, U$1.VSS2, U$1.VSSA, U1.GND*6, U2.RES, U3.GND
- net LED_HID: now also D5.C, U1.LED_HID; no longer D3.C, U$1.LED_HID
- net LED_MSD: now also D4.C, U1.LED_MSD; no longer D2.C, U$1.LED_MSD
- net LED_UART: now also D6.C, U1.LED_UART; no longer D4.C, U$1.LED_UART
- net N$1: now also D4.A, R25.1; no longer D2.A, R2.1
- net N$10: now also R2.1, U1.NRESET_FB_BL; no longer R13.1, U$1.NRESET_FB_BL
- net N$11: now also R11.1, U1.SLEEP_NREQ; no longer R19.1, U$1.SLEEP_NREQ
- net N$13: now also TP5.1, U1.XTALIN, U2.1; no longer TP2.1, U$1.XTALIN, Y1.2
- net N$14: now also C14.2, U3.XI, Y1.2; no longer C13.2, U1.XI, Y2.2
- net N$15: now also C15.2, U3.XO, Y1.1; no longer C14.2, U1.XO, Y2.1
- net N$16: now also C10.1, U1.XTALOUT, U2.2; no longer C8.1, U$1.XTALOUT, Y1.1
- net N$17: now also R12.1, TP3.1, U1.TGT_TX; no longer R25.1, TP16.1, U$1.TGT_TX
- net N$18: now also R13.1, TP4.1, U1.TGT_RX; no longer R26.1, TP15.1, U$1.TGT_RX
- net N$19: now also R10.1, U1.WAKE_NREQ; no longer R18.1, U$1.WAKE_NREQ
- net N$2: now also D5.A, R26.1; no longer D3.A, R3.1
- net N$20: now also R22.2, TP2.1, U3.~BOOT(MOSI5/RX1/32KHZ); no longer R27.2, TP17.1, U1.~BOOT(MOSI5/RX1/32KHZ)
- net N$21: now also D2.A, J1.2, TP12.1; no longer D6.A, J2.2, TP10.1
- net N$22: now also R9.1, U1.TGT_NRESET; no longer R20.2, U$1.TGT_NRESET
- net N$23: now also R4.1, U1.TGT_SWCLK; no longer R22.1, TP12.1, U$1.TGT_SWCLK
- net N$24: now also R5.1, U1.TGT_SWDIO; no longer R23.1, TP13.1, U$1.TGT_SWDIO
- net N$25: now also R6.1, U1.TGT_SWO; no longer R24.1, TP14.1, U$1.TGT_SWO
- net N$3: now also D6.A, R27.1; no longer D4.A, R4.1
- net N$4: now also J2.CC2, R7.2; no longer J1.CC2, R5.2
- net N$5: now also J2.CC1, R8.2; no longer J1.CC1, R6.2
- net N$7: now also D7.A, R28.1; no longer D1.A, R10.1
- net N$8: now also D3.4, R23.1; no longer D5.4, R8.1
- net N$9: now also D3.6, R29.1; no longer D5.6, R7.1
- net PDM_CLK: now also U3.~AD12(PDMCLK/TX1); no longer U1.~AD12(PDMCLK/TX1)
- net PDM_DATA: now also U3.~AD11(PDMDATA); no longer U1.~AD11(PDMDATA)
- net SCL: now also J8.4, R20.1, U3.(SCL1/SCK1/TX1/SCCLK)D8; no longer J5.4, R29.1, U1.(SCL1/SCK1/TX1/SCCLK)D8
- net SCL_INTERNAL: now also U3.(SCL2/SCK2)~D27, U5.SCL/SPC; no longer U1.(SCL2/SCK2)~D27, U2.SCL/SPC
- net SDA: now also J8.3, R21.1, U3.(SDA1/MISO1/RX1/SCCIO)D9; no longer J5.3, R28.1, U1.(SDA1/MISO1/RX1/SCCIO)D9
- net SDA_INTERNAL: now also U3.(SDA2/MISO2/RX1)~D25, U5.SDA/SDI/SDO; no longer U1.(SDA2/MISO2/RX1)~D25, U2.SDA/SDI/SDO
- net TCLK: now also J4.SWDCLK/TCK, R18.1, U1.NC4; no longer J3.SWDCLK/TCK, R17.1, TP6.1, U$1.NC4
- net TDI: now also J4.NC/TDI, R17.1, U1.NC5; no longer J3.NC/TDI, R16.1, TP5.1, U$1.NC5
- net TDO: now also J4.SWO/TDO, R16.1, U1.NC6; no longer J3.SWO/TDO, R15.1, TP4.1, U$1.NC6
- net TGT_RX: now also R13.2, U3.~D48(TX0/SCL5/SCK5); no longer R26.2, U1.~D48(TX0/SCL5/SCK5)
- net TGT_SWCLK: now also J3.SWDCLK, R4.2, U3.D20(SWDCK/TX1); no longer J4.SWDCLK, R22.2, U1.D20(SWDCK/TX1)
- net TGT_SWDIO: now also J3.SWDIO, R5.2, U3.D21(SWDIO/RX1/SCCRST); no longer J4.SWDIO, R23.2, U1.D21(SWDIO/RX1/SCCRST)
- net TGT_SWO: now also J3.SWO, R6.2, U3.(PDMCLK/SWO)~D22; no longer J4.SWO, R24.2, U1.(PDMCLK/SWO)~D22
- net TGT_TX: now also R12.2, U3.~D49(RX0/SDA5/MISO5); no longer R25.2, U1.~D49(RX0/SDA5/MISO5)
- net TMS: now also J4.SWDIO/TMS, R15.1, U1.NC7; no longer J3.SWDIO/TMS, R14.1, TP3.1, U$1.NC7
- net USB_D+_P: now also R23.2, U1.USB_D+; no longer R8.2, U$1.USB_D+
- net USB_D+_R: now also D3.3, J2.D+; no longer D5.3, J1.D+
- net USB_D-_P: now also R29.2, U1.USB_D-; no longer R7.2, U$1.USB_D-
- net USB_D-_R: now also D3.1, J2.D-; no longer D5.1, J1.D-
- net VBUS_IF: now also D3.5, J2.VBUS, R24.1; no longer J1.VBUS
- net VBUS_IF2: now also C12.1, C13.1, R14.2, R24.2, U1.VREGIN; no longer C2.1, C3.1, R12.2, R9.2, U$1.VREGIN
- net VDD: now also C18.1, C19.1, C2.1, C3.1, C4.1, D1.C, D2.C, J3.VCC, J5.7, J8.2, R20.2, R3.2, TP10.1, U3.VDD*2, U4.IN, U5.CS, U5.SDO/SA0, U5.VDD, U5.VDD_IO; no longer C10.1, C11.1, C12.1, C16.1, C22.1, D6.C, D7.C, J4.VCC, J5.2, J8.7, R28.2, R29.2, TP9.1, U1.VDD*2, U2.CS, U2.SDO/SA0, U2.VDD, U2.VDD_IO, U3.IN
Other:
- moved on the sheet: C10, C11, C12, C13, C14, C15, C16, C17, C2, C20, C21, C3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
