File: hardware/Artembed.brd (EAGLE design)
At the start: 160 x 100 mm, 90 parts, among them J3 CORTEX_JTAG_DEBUG_MINIMUM_PTH, J4 CORTEX_JTAG_DEBUG_PTH_NS, J7 CAMERA-HIMAX, U1 DAPLINK_KL26Z, U2 16MHz, U3 ARTEMIS_MODULESMD, U4 1.8V, U5 LIS2DH12, Y1 32.768kHz

Commit message: progress
Parts:
- moved J7 2.54 mm to (39.4, 2.54)
- moved J9 1.27 mm to (29.2, 16.5)
- moved J5 0.63 mm to (27.9, 18.4)
