File: hardware/small_form_factor/Artembed_SMALL.brd (EAGLE design)
At the start: 160 x 100 mm, 88 parts, among them J3 CORTEX_JTAG_DEBUG_MINIMUM_PTH, J4 CORTEX_JTAG_DEBUG_PTH_NS, J7 CAMERA-HIMAX, U1 DAPLINK_KL26Z, U2 16MHz, U3 ARTEMIS_MODULESMD, U4 1.8V, U5 LIS2DH12, Y1 32.768kHz

Commit message: Back up small form factor
Moving to a more prototyping friendly large form factor for now
Parts:
- moved TP1 68.9 mm to (31.8, 12.4)
- moved U4 64.3 mm to (35.2, 13.0), flipped to the bottom
- moved R30 63.9 mm to (35.2, 10.2), flipped to the bottom
- moved C16 62.7 mm to (37.3, 13.0), flipped to the bottom
- moved C19 58.6 mm to (38.9, 13.0), flipped to the bottom, turned to 90 degrees
- moved R22 57.6 mm to (45.0, 13.0), turned to 90 degrees
- moved TP2 56.2 mm to (46.5, 13.7)
- moved Y1 53.8 mm to (34.4, 4.06)
- moved C14 51.6 mm to (34.0, 1.40), flipped to the top
- moved C21 43.6 mm to (89.0, 43.8)
- moved JP1 27.4 mm to (57.4, 14.5), flipped to the bottom, turned to 90 degrees
- moved R6 17.2 mm to (40.4, 13.0), turned to 90 degrees
- moved R4 14.8 mm to (41.9, 13.0), turned to 90 degrees
- moved R5 10.5 mm to (43.4, 13.0), turned to 90 degrees
- moved C15 8.89 mm to (68.6, 32.0), flipped to the top
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Routing:
- net TGT_SWCLK: track 0.00 -> 9.13 mm, vias 0 -> 1
- net TGT_SWO: track 0.00 -> 7.62 mm
- net VDD: track 22.8 -> 29.6 mm, vias 2 -> 3
- net 1.8V: track 0.00 -> 6.73 mm
- net N$20: track 0.00 -> 5.17 mm, vias 0 -> 1
- net N$14: track 0.00 -> 4.81 mm
- net SCL_INTERNAL: track 19.5 -> 15.3 mm, vias 1 -> 2
- net TGT_SWDIO: track 0.00 -> 4.04 mm
- net N$15: track 0.00 -> 3.97 mm
- net GND: track 29.8 -> 33.0 mm, vias 7 -> 8
- net TGT_TX: track 0.00 -> 2.66 mm, vias 0 -> 1
- net CAMERA_D2: track 0.00 -> 1.80 mm, vias 0 -> 1
- net SDA: track 13.5 -> 15.2 mm, vias 1 -> 2
- net SDA_INTERNAL: track 14.4 -> 12.9 mm
- net CAMERA_D1: track 0.00 -> 1.08 mm, vias 0 -> 1
