File: hardware/Production/ArtemisDevKit-Panel.brd (EAGLE design)
At the start: 116.6 x 181.4 mm, 925 parts, among them J1 USB, J10 SMD, J11 SMD, J12 PTH, J13 USB, J14 PTH, J15 CORTEX_JTAG_DEBUG_MINIMUM_PTH, J16 CORTEX_JTAG_DEBUG_PTH, J17 QWIIC_RIGHT_ANGLE, J18 CAMERA-HIMAXBOTTOM-CONTACT, J19 SMD, J2 CORTEX_JTAG_DEBUG_MINIMUM_PTH, J20 PTH, J21 PTH, J22 PTH, J23 PTH, J24 PTH, J25 PTH, J26 PTH, J27 PTH, J28 PTH, J29 PTH, J3 CORTEX_JTAG_DEBUG_PTH, J30 PTH, J31 PTH, J32 PTH, J33 1X04_SMD_STRAIGHT_COMBO, J34 1X04_SMD_STRAIGHT_COMBO, J35 SMD, J36 SMD, J37 USB, J38 CORTEX_JTAG_DEBUG_MINIMUM_PTH, J39 CORTEX_JTAG_DEBUG_PTH, J4 SMD, J40 QWIIC_RIGHT_ANGLE, J41 CAMERA-HIMAXBOTTOM-CONTACT, J42 SMD, J43 PTH, J44 PTH, J45 PTH, J46 PTH, J47 PTH, J48 PTH, J49 PTH, J5 1X04_SMD_STRAIGHT_COMBO, J50 PTH, J51 1X04_SMD_STRAIGHT_COMBO, J52 1X04_SMD_STRAIGHT_COMBO, J53 SMD, J54 SMD, J55 USB, J56 CORTEX_JTAG_DEBUG_MINIMUM_PTH, J57 CORTEX_JTAG_DEBUG_PTH, J58 QWIIC_RIGHT_ANGLE, J59 CAMERA-HIMAXBOTTOM-CONTACT, J6 QWIIC_RIGHT_ANGLE, J60 SMD, J61 PTH, J62 PTH, J63 PTH, J64 PTH, J65 PTH, J66 PTH, J67 PTH, J68 PTH, J69 1X04_SMD_STRAIGHT_COMBO, J7 CAMERA-HIMAXBOTTOM-CONTACT, J70 1X04_SMD_STRAIGHT_COMBO, J71 SMD, J72 SMD, J8 PTH, J9 1X04_SMD_STRAIGHT_COMBO, U1 DAPLINK_KL26Z128VFM4, U10 DAPLINK_KL26Z128VFM4, U11 ARTEMIS_MODULESMD, U12 LIS2DH12, U13 AP2127K-1.8V, U14 3.3V, U15 DAPLINK_KL26Z128VFM4, U16 ARTEMIS_MODULESMD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

Commit message: generate gerbers
Parts:
- removed J65, J66, J67, J68: PTH, SparkFun-Connectors:1X12_NO_SILK
- removed J69, J70: 1X04_SMD_STRAIGHT_COMBO, SparkFun-Connectors:1X04_SMD_VERTICAL_COMBO
- removed J71, J72: SMD, SparkFun-Connectors:1X08_SMD_COMBINED
- J10: value SMD -> USB; device SparkFun-Connectors:1X08_SMD_COMBINED -> SparkFun-Connectors:USB-C-16P
- J11: value SMD -> CORTEX_JTAG_DEBUG_MINIMUM_PTH; device SparkFun-Connectors:1X08_SMD_COMBINED -> SparkFun-Connectors:2X5-PTH-1.27MM
- J13: value USB -> CORTEX_JTAG_DEBUG_PTH; device SparkFun-Connectors:USB-C-16P -> SparkFun-Connectors:2X5-PTH-1.27MM
- J15: value CORTEX_JTAG_DEBUG_MINIMUM_PTH -> QWIIC_RIGHT_ANGLE; device SparkFun-Connectors:2X5-PTH-1.27MM -> SparkFun-Connectors:JST04_1MM_RA
- J16: value CORTEX_JTAG_DEBUG_PTH -> CAMERA-HIMAXBOTTOM-CONTACT; device SparkFun-Connectors:2X5-PTH-1.27MM -> SparkFun-Connectors:FPC-24-AMPHENOL-SFV24R-1STE1HLF
- J17: value QWIIC_RIGHT_ANGLE -> SMD; device SparkFun-Connectors:JST04_1MM_RA -> SparkFun-Connectors:1X08_SMD_COMBINED
- J18: value CAMERA-HIMAXBOTTOM-CONTACT -> PTH; device SparkFun-Connectors:FPC-24-AMPHENOL-SFV24R-1STE1HLF -> SparkFun-Connectors:1X08_NO_SILK
- J19: value SMD -> PTH; device SparkFun-Connectors:1X08_SMD_COMBINED -> SparkFun-Connectors:1X08_NO_SILK
- J20, J21, J43, J44, J61, J62: device SparkFun-Connectors:1X08_NO_SILK -> SparkFun-Connectors:1X12_NO_SILK
- J31, J32, J47, J48, J63, J64: value PTH -> (none); device SparkFun-Connectors:1X12_NO_SILK -> SparkFun-Connectors:1X12_SMD_COMBINED
- J33: value 1X04_SMD_STRAIGHT_COMBO -> USB; device SparkFun-Connectors:1X04_SMD_VERTICAL_COMBO -> SparkFun-Connectors:USB-C-16P
- J34: value 1X04_SMD_STRAIGHT_COMBO -> CORTEX_JTAG_DEBUG_MINIMUM_PTH; device SparkFun-Connectors:1X04_SMD_VERTICAL_COMBO -> SparkFun-Connectors:2X5-PTH-1.27MM
- J35: value SMD -> CORTEX_JTAG_DEBUG_PTH; device SparkFun-Connectors:1X08_SMD_COMBINED -> SparkFun-Connectors:2X5-PTH-1.27MM
- J36: value SMD -> QWIIC_RIGHT_ANGLE; device SparkFun-Connectors:1X08_SMD_COMBINED -> SparkFun-Connectors:JST04_1MM_RA
- J37: value USB -> CAMERA-HIMAXBOTTOM-CONTACT; device SparkFun-Connectors:USB-C-16P -> SparkFun-Connectors:FPC-24-AMPHENOL-SFV24R-1STE1HLF
- J38: value CORTEX_JTAG_DEBUG_MINIMUM_PTH -> SMD; device SparkFun-Connectors:2X5-PTH-1.27MM -> SparkFun-Connectors:1X08_SMD_COMBINED
- J39: value CORTEX_JTAG_DEBUG_PTH -> PTH; device SparkFun-Connectors:2X5-PTH-1.27MM -> SparkFun-Connectors:1X08_NO_SILK
- J40: value QWIIC_RIGHT_ANGLE -> PTH; device SparkFun-Connectors:JST04_1MM_RA -> SparkFun-Connectors:1X08_NO_SILK
- J41, J59: value CAMERA-HIMAXBOTTOM-CONTACT -> PTH; device SparkFun-Connectors:FPC-24-AMPHENOL-SFV24R-1STE1HLF -> SparkFun-Connectors:1X12_NO_SILK
- J42, J60: value SMD -> PTH; device SparkFun-Connectors:1X08_SMD_COMBINED -> SparkFun-Connectors:1X12_NO_SILK
- J49: value PTH -> USB; device SparkFun-Connectors:1X12_NO_SILK -> SparkFun-Connectors:USB-C-16P
- J5, J9: value 1X04_SMD_STRAIGHT_COMBO -> (none); device SparkFun-Connectors:1X04_SMD_VERTICAL_COMBO -> SparkFun-Connectors:1X12_SMD_COMBINED
- J50: value PTH -> CORTEX_JTAG_DEBUG_MINIMUM_PTH; device SparkFun-Connectors:1X12_NO_SILK -> SparkFun-Connectors:2X5-PTH-1.27MM
- J51: value 1X04_SMD_STRAIGHT_COMBO -> CORTEX_JTAG_DEBUG_PTH; device SparkFun-Connectors:1X04_SMD_VERTICAL_COMBO -> SparkFun-Connectors:2X5-PTH-1.27MM
- J52: value 1X04_SMD_STRAIGHT_COMBO -> QWIIC_RIGHT_ANGLE; device SparkFun-Connectors:1X04_SMD_VERTICAL_COMBO -> SparkFun-Connectors:JST04_1MM_RA
- J53: value SMD -> CAMERA-HIMAXBOTTOM-CONTACT; device SparkFun-Connectors:1X08_SMD_COMBINED -> SparkFun-Connectors:FPC-24-AMPHENOL-SFV24R-1STE1HLF
- J55: value USB -> PTH; device SparkFun-Connectors:USB-C-16P -> SparkFun-Connectors:1X08_NO_SILK
- J56: value CORTEX_JTAG_DEBUG_MINIMUM_PTH -> PTH; device SparkFun-Connectors:2X5-PTH-1.27MM -> SparkFun-Connectors:1X08_NO_SILK
- J57: value CORTEX_JTAG_DEBUG_PTH -> PTH; device SparkFun-Connectors:2X5-PTH-1.27MM -> SparkFun-Connectors:1X12_NO_SILK
- J58: value QWIIC_RIGHT_ANGLE -> PTH; device SparkFun-Connectors:JST04_1MM_RA -> SparkFun-Connectors:1X12_NO_SILK
- moved J52 95.1 mm to (5.08, 147.6), turned to 270 degrees
- moved J39 91.5 mm to (92.1, 110.2)
- moved J49 89.1 mm to (6.35, 134.9), turned to 270 degrees
- moved J36 87.5 mm to (5.08, 109.0), turned to 270 degrees
- moved J55 86.9 mm to (92.1, 148.8)
- moved J40 85.1 mm to (90.2, 110.2)
- moved J34 82.5 mm to (21.6, 108.4), turned to 270 degrees
- moved J17 81.3 mm to (86.4, 71.6)
- moved J11 75.9 mm to (21.6, 69.8), turned to 270 degrees
- moved J57 75.1 mm to (78.7, 119.6), turned to 180 degrees
- moved J33 71.3 mm to (6.35, 96.3), turned to 270 degrees
- moved J51 70.1 mm to (3.81, 124.7), turned to 270 degrees
- moved J56 68.6 mm to (90.2, 148.8)
- moved J38 64.7 mm to (86.4, 110.2)
- moved J54 64.0 mm to (86.4, 148.8), turned to 270 degrees
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Connections:
- net !INTFC_RST1: now also J13.10; no longer J16.10
- net !INTFC_RST2: now also J35.10; no longer J39.10
- net !INTFC_RST3: now also J51.10; no longer J57.10
- net !TGT_RST1: now also J11.10; no longer J15.10
- net !TGT_RST2: now also J34.10; no longer J38.10
- net !TGT_RST3: now also J50.10; no longer J56.10
- net 1.8V1: now also J16.10, J17.7, J17.7@2, J17.8, J17.8@2, J18.7, J18.8; no longer J18.10, J19.7@2, J19.8@2, J20.7, J20.8, J21.7, J21.8
- net 1.8V2: now also J37.10, J38.7, J38.7@2, J38.8, J38.8@2, J39.7, J39.8, J40.7, J40.8; no longer J41.10, J42.7, J42.7@2, J42.8, J42.8@2, J43.7, J43.8, J44.7, J44.8
- net 1.8V3: now also J53.10, J54.7, J54.7@2, J54.8, J54.8@2, J55.7, J55.8, J56.7, J56.8; no longer J59.10, J60.7, J60.7@2, J60.8, J60.8@2, J61.7, J61.8, J62.7, J62.8
- net 3.3V1: now also J11.1, J13.1, J15.2, J16.11, J16.4, J17.5, J17.5@2, J17.6, J17.6@2, J18.5, J18.6; no longer J15.1, J16.1, J17.2, J18.11, J18.4, J19.5@2, J19.6@2, J20.5, J20.6, J21.5, J21.6
- net 3.3V2: now also J34.1, J35.1, J36.2, J37.11, J37.4, J38.5, J38.5@2, J38.6, J38.6@2, J39.5, J39.6, J40.5, J40.6; no longer J38.1, J39.1, J40.2, J41.11, J41.4, J42.5, J42.5@2, J42.6, J42.6@2, J43.5, J43.6, J44.5, J44.6
- net 3.3V3: now also J50.1, J51.1, J52.2, J53.11, J53.4, J54.5, J54.5@2, J54.6, J54.6@2, J55.5, J55.6, J56.5, J56.6; no longer J56.1, J57.1, J58.2, J59.11, J59.4, J60.5, J60.5@2, J60.6, J60.6@2, J61.5, J61.6, J62.5, J62.6
- net CAMERA_D10: now also J16.12; no longer J18.12
- net CAMERA_D11: now also J16.20; no longer J18.20
- net CAMERA_D12: now also J16.19; no longer J18.19
- net CAMERA_D13: now also J16.13; no longer J18.13
- net CAMERA_D14: now also J16.14; no longer J18.14
- net CAMERA_D15: now also J16.9; no longer J18.9
- net CAMERA_D16: now also J37.3; no longer J41.3
- net CAMERA_D17: now also J37.5; no longer J41.5
- net CAMERA_D18: now also J37.12; no longer J41.12
- net CAMERA_D19: now also J37.20; no longer J41.20
- net CAMERA_D20: now also J37.19; no longer J41.19
- net CAMERA_D21: now also J37.13; no longer J41.13
- net CAMERA_D22: now also J37.14; no longer J41.14
- net CAMERA_D23: now also J37.9; no longer J41.9
- net CAMERA_D24: now also J53.3; no longer J59.3
- net CAMERA_D25: now also J53.5; no longer J59.5
- net CAMERA_D26: now also J53.12; no longer J59.12
- net CAMERA_D27: now also J53.20; no longer J59.20
- net CAMERA_D28: now also J53.19; no longer J59.19
- net CAMERA_D29: now also J53.13; no longer J59.13
- net CAMERA_D30: now also J53.14; no longer J59.14
- net CAMERA_D31: now also J53.9; no longer J59.9
- net CAMERA_D8: now also J16.3; no longer J18.3
- net CAMERA_D9: now also J16.5; no longer J18.5
- net CAMERA_HSYNC1: now also J16.16; no longer J18.16
- net CAMERA_HSYNC2: now also J37.16; no longer J41.16
- net CAMERA_HSYNC3: now also J53.16; no longer J59.16
- net CAMERA_INT1: now also J16.18; no longer J18.18
- net CAMERA_INT2: now also J37.18; no longer J41.18
- net CAMERA_INT3: now also J53.18; no longer J59.18
- net CAMERA_MCLK1: now also J16.8; no longer J18.8
- net CAMERA_MCLK2: now also J37.8; no longer J41.8
- net CAMERA_MCLK3: now also J53.8; no longer J59.8
- net CAMERA_PCLK1: now also J16.17; no longer J18.17
- net CAMERA_PCLK2: now also J37.17; no longer J41.17
- net CAMERA_PCLK3: now also J53.17; no longer J59.17
- net CAMERA_TRIG1: now also J16.7; no longer J18.7
- net CAMERA_TRIG2: now also J37.7; no longer J41.7
- net CAMERA_TRIG3: now also J53.7; no longer J59.7
- net CAMERA_VSYNC1: now also J16.6; no longer J18.6
- net CAMERA_VSYNC2: now also J37.6; no longer J41.6
- net CAMERA_VSYNC3: now also J53.6; no longer J59.6
- net D1: now also J21.3, J30.3, J31.3, J31.3@2; no longer J28.3, J32.3, J35.3, J35.3@2
- net D10: now also J20.4, J29.4, J32.4, J32.4@2; no longer J27.4, J31.4, J34.4, J34.4-2
- net D11: now also J20.12, J29.12, J32.12, J32.12@2; no longer J27.12, J31.12, J36.8, J36.8@2
- net D12: now also J21.6, J30.6, J31.6, J31.6@2; no longer J28.6, J32.6, J35.6, J35.6@2
- net D13: now also J9.5, J9.5@2; no longer J11.1, J11.1@2
- net D14: now also J21.4, J30.4, J31.4, J31.4@2; no longer J28.4, J32.4, J35.4, J35.4@2
- net D15: now also J21.9, J30.9, J31.9, J31.9@2; no longer J28.9, J32.9, J33.1, J33.1-2
- net D16: now also J5.12, J5.12@2; no longer J5.4, J5.4-2
- net D17: now also J20.5, J29.5, J32.5, J32.5@2; no longer J27.5, J31.5, J36.1, J36.1@2
- net D18: now also J21.12, J30.12, J31.12, J31.12@2; no longer J28.12, J32.12, J33.4, J33.4-2
- net D19: now also J20.8, J29.8, J32.8, J32.8@2; no longer J27.8, J31.8, J36.4, J36.4@2
- net D2: now also J21.2, J30.2, J31.2, J31.2@2; no longer J28.2, J32.2, J35.2, J35.2@2
- net D20: now also J21.11, J30.11, J31.11, J31.11@2; no longer J28.11, J32.11, J33.3, J33.3-2
- net D21: now also J20.7, J29.7, J32.7, J32.7@2; no longer J27.7, J31.7, J36.3, J36.3@2
- net D22: now also J20.6, J29.6, J32.6, J32.6@2; no longer J27.6, J31.6, J36.2, J36.2@2
- net D23: now also J20.9, J29.9, J32.9, J32.9@2; no longer J27.9, J31.9, J36.5, J36.5@2
- net D23_LED: now also J9.3@2; no longer J9.3-2
- net D23_LED1: now also J20.3, J29.3, J32.3, J32.3@2; no longer J27.3, J31.3, J34.3, J34.3-2
- net D23_LED2: now also J41.3, J48.3, J48.3@2; no longer J49.3, J52.3, J52.3-2
- net D23_LED3: now also J57.3, J61.3, J64.3, J64.3@2; no longer J63.3, J67.3, J70.3, J70.3-2
- net D24: now also J9.1@2; no longer J9.1-2
- net D25: now also J9.11, J9.11@2; no longer J11.7, J11.7@2
- net D26: now also J9.10, J9.10@2; no longer J11.6, J11.6@2
- net D27: now also J9.4@2; no longer J9.4-2
- net D28: now also J9.12, J9.12@2; no longer J11.8, J11.8@2
- net D29: now also J9.8, J9.8@2; no longer J11.4, J11.4@2
- net D3: now also J21.1, J30.1, J31.1, J31.1@2; no longer J28.1, J32.1, J35.1, J35.1@2
- net D30: now also J20.1, J29.1, J32.1, J32.1@2; no longer J27.1, J31.1, J34.1, J34.1-2
- net D31: now also J5.11, J5.11@2; no longer J5.3, J5.3-2
- net D32: now also J9.7, J9.7@2; no longer J11.3, J11.3@2
- net D33: now also J9.6, J9.6@2; no longer J11.2, J11.2@2
- net D34: now also J9.9, J9.9@2; no longer J11.5, J11.5@2
- net D35: now also J9.2@2; no longer J9.2-2
- net D36: now also J5.6, J5.6@2; no longer J10.6, J10.6@2
- net D37: now also J5.4, J5.4@2; no longer J10.4, J10.4@2
- net D38: now also J5.5, J5.5@2; no longer J10.5, J10.5@2
- net D39: now also J5.1, J5.1@2; no longer J10.1, J10.1@2
- net D4: now also J21.5, J30.5, J31.5, J31.5@2; no longer J28.5, J32.5, J35.5, J35.5@2
- net D40: now also J5.2, J5.2@2; no longer J10.2, J10.2@2
- net D41: now also J5.10, J5.10@2; no longer J5.2, J5.2-2
- net D42: now also J5.7, J5.7@2; no longer J10.7, J10.7@2
- net D43: now also J5.8, J5.8@2; no longer J10.8, J10.8@2
- net D44: now also J5.3, J5.3@2; no longer J10.3, J10.3@2
- net D45: now also J5.9, J5.9@2; no longer J5.1, J5.1-2
- net D46: now also J20.2, J29.2, J32.2, J32.2@2; no longer J27.2, J31.2, J34.2, J34.2-2
- net D47: now also J42.3, J47.3, J47.3@2; no longer J50.3, J53.3, J53.3@2
- net D48: now also J42.2, J47.2, J47.2@2; no longer J50.2, J53.2, J53.2@2
- net D49: now also J42.1, J47.1, J47.1@2; no longer J50.1, J53.1, J53.1@2
- net D5: now also J21.8, J30.8, J31.8, J31.8@2; no longer J28.8, J32.8, J35.8, J35.8@2
- net D50: now also J42.5, J47.5, J47.5@2; no longer J50.5, J53.5, J53.5@2
- net D51: now also J42.8, J47.8, J47.8@2; no longer J50.8, J53.8, J53.8@2
- net D52: now also J42.7, J47.7, J47.7@2; no longer J50.7, J53.7, J53.7@2
- net D53: now also J42.10, J47.10, J47.10@2; no longer J50.10, J51.2, J51.2-2
- net D54: now also J41.11, J48.11, J48.11@2; no longer J49.11, J54.7, J54.7@2
- net D55: now also J41.10, J48.10, J48.10@2; no longer J49.10, J54.6, J54.6@2
- net D56: now also J41.4, J48.4, J48.4@2; no longer J49.4, J52.4, J52.4-2
- net D57: now also J41.12, J48.12, J48.12@2; no longer J49.12, J54.8, J54.8@2
- net D58: now also J42.6, J47.6, J47.6@2; no longer J50.6, J53.6, J53.6@2
- net D59: now also J42.4, J47.4, J47.4@2; no longer J50.4, J53.4, J53.4@2
- net D6: now also J21.7, J30.7, J31.7, J31.7@2; no longer J28.7, J32.7, J35.7, J35.7@2
- net D60: now also J42.9, J47.9, J47.9@2; no longer J50.9, J51.1, J51.1-2
- net D61: now also J41.5, J48.5, J48.5@2; no longer J49.5, J54.1, J54.1@2
- net D62: now also J42.12, J47.12, J47.12@2; no longer J50.12, J51.4, J51.4-2
- net D63: now also J41.8, J48.8, J48.8@2; no longer J49.8, J54.4, J54.4@2
- net D64: now also J42.11, J47.11, J47.11@2; no longer J50.11, J51.3, J51.3-2
- net D65: now also J41.7, J48.7, J48.7@2; no longer J49.7, J54.3, J54.3@2
- net D66: now also J41.6, J48.6, J48.6@2; no longer J49.6, J54.2, J54.2@2
- net D67: now also J41.9, J48.9, J48.9@2; no longer J49.9, J54.5, J54.5@2
- net D68: now also J41.1, J48.1, J48.1@2; no longer J49.1, J52.1, J52.1-2
- net D69: now also J41.2, J48.2, J48.2@2; no longer J49.2, J52.2, J52.2-2
- net D7: now also J21.10, J30.10, J31.10, J31.10@2; no longer J28.10, J32.10, J33.2, J33.2-2
- net D70: now also J58.3, J62.3, J63.3, J63.3@2; no longer J64.3, J68.3, J71.3, J71.3@2
- net D71: now also J58.2, J62.2, J63.2, J63.2@2; no longer J64.2, J68.2, J71.2, J71.2@2
- net D72: now also J58.1, J62.1, J63.1, J63.1@2; no longer J64.1, J68.1, J71.1, J71.1@2
- net D73: now also J58.5, J62.5, J63.5, J63.5@2; no longer J64.5, J68.5, J71.5, J71.5@2
- net D74: now also J58.8, J62.8, J63.8, J63.8@2; no longer J64.8, J68.8, J71.8, J71.8@2
- net D75: now also J58.7, J62.7, J63.7, J63.7@2; no longer J64.7, J68.7, J71.7, J71.7@2
- net D76: now also J58.10, J62.10, J63.10, J63.10@2; no longer J64.10, J68.10, J69.2, J69.2-2
- net D77: now also J57.11, J61.11, J64.11, J64.11@2; no longer J63.11, J67.11, J72.7, J72.7@2
- net D78: now also J57.10, J61.10, J64.10, J64.10@2; no longer J63.10, J67.10, J72.6, J72.6@2
- net D79: now also J57.4, J61.4, J64.4, J64.4@2; no longer J63.4, J67.4, J70.4, J70.4-2
- net D8: now also J20.11, J29.11, J32.11, J32.11@2; no longer J27.11, J31.11, J36.7, J36.7@2
- net D80: now also J57.12, J61.12, J64.12, J64.12@2; no longer J63.12, J67.12, J72.8, J72.8@2
- net D81: now also J58.6, J62.6, J63.6, J63.6@2; no longer J64.6, J68.6, J71.6, J71.6@2
- net D82: now also J58.4, J62.4, J63.4, J63.4@2; no longer J64.4, J68.4, J71.4, J71.4@2
- net D83: now also J58.9, J62.9, J63.9, J63.9@2; no longer J64.9, J68.9, J69.1, J69.1-2
- net D84: now also J57.5, J61.5, J64.5, J64.5@2; no longer J63.5, J67.5, J72.1, J72.1@2
- net D85: now also J58.12, J62.12, J63.12, J63.12@2; no longer J64.12, J68.12, J69.4, J69.4-2
- net D86: now also J57.8, J61.8, J64.8, J64.8@2; no longer J63.8, J67.8, J72.4, J72.4@2
- net D87: now also J58.11, J62.11, J63.11, J63.11@2; no longer J64.11, J68.11, J69.3, J69.3-2
- net D88: now also J57.7, J61.7, J64.7, J64.7@2; no longer J63.7, J67.7, J72.3, J72.3@2
- net D89: now also J57.6, J61.6, J64.6, J64.6@2; no longer J63.6, J67.6, J72.2, J72.2@2
- net D9: now also J20.10, J29.10, J32.10, J32.10@2; no longer J27.10, J31.10, J36.6, J36.6@2
- net D90: now also J57.9, J61.9, J64.9, J64.9@2; no longer J63.9, J67.9, J72.5, J72.5@2
- net D91: now also J57.1, J61.1, J64.1, J64.1@2; no longer J63.1, J67.1, J70.1, J70.1-2
- net D92: now also J57.2, J61.2, J64.2, J64.2@2; no longer J63.2, J67.2, J70.2, J70.2-2
- net GND1: now also J10.GND, J10.GND2, J11.3, J11.5, J11.9, J13.3, J13.5, J13.9, J15.1, J16.15, J16.2, J17.1@2, J17.2, J17.2@2, J18.1, J27.1, J27.10, J27.11, J27.12, J27.2, J27.3, J27.4, J27.5, J27.6, J27.7, J27.8, J27.9, J28.1, J28.10, J28.11, J28.12, J28.2, J28.3, J28.4, J28.5, J28.6, J28.7, J28.8, J28.9; no longer J13.GND, J13.GND2, J15.3, J15.5, J15.9, J16.3, J16.5, J16.9, J18.15, J19.1@2, J19.2@2, J20.1, J20.2, J21.1, J21.2, J29.1, J29.10, J29.11, J29.12, J29.2, J29.3, J29.4, J29.5, J29.6, J29.7, J29.8, J29.9, J30.1, J30.10, J30.11, J30.12, J30.2, J30.3, J30.4, J30.5, J30.6, J30.7, J30.8, J30.9
- net GND2: now also J33.GND, J33.GND2, J34.3, J34.5, J34.9, J35.3, J35.5, J35.9, J36.1, J37.15, J37.2, J38.1, J38.1@2, J38.2, J38.2@2, J39.1, J39.2, J40.2, J43.10, J43.11, J43.12, J43.3, J43.4, J43.5, J43.6, J43.7, J43.8, J43.9, J44.10, J44.11, J44.12, J44.3, J44.4, J44.5, J44.6, J44.7, J44.8, J44.9; no longer J37.GND, J37.GND2, J38.3, J38.5, J38.9, J39.3, J39.5, J39.9, J41.15, J41.2, J42.1, J42.1@2, J42.2, J42.2@2, J47.1, J47.10, J47.11, J47.12, J47.2, J47.3, J47.4, J47.5, J47.6, J47.7, J47.8, J47.9, J48.1, J48.10, J48.11, J48.12, J48.2, J48.3, J48.4, J48.5, J48.6, J48.7, J48.8, J48.9
- net GND3: now also J49.GND, J49.GND2, J50.3, J50.5, J50.9, J51.3, J51.5, J51.9, J52.1, J53.15, J53.2, J54.1, J54.1@2, J54.2, J54.2@2, J55.1, J55.2, J56.1, J56.2, J59.1, J59.10, J59.11, J59.12, J59.3, J59.4, J59.5, J59.6, J59.7, J59.8, J59.9, J60.10, J60.11, J60.12, J60.3, J60.4, J60.5, J60.6, J60.7, J60.8, J60.9; no longer J55.GND, J55.GND2, J56.3, J56.5, J56.9, J57.3, J57.5, J57.9, J58.1, J59.15, J60.1@2, J60.2@2, J61.1, J61.2, J62.1, J62.2, J65.1, J65.10, J65.11, J65.12, J65.2, J65.3, J65.4, J65.5, J65.6, J65.7, J65.8, J65.9, J66.1, J66.10, J66.11, J66.12, J66.2, J66.3, J66.4, J66.5, J66.6, J66.7, J66.8, J66.9
- net INTFC_NC1: now also J13.6; no longer J16.6
- net INTFC_NC2: now also J13.8; no longer J16.8
- net INTFC_NC3: now also J35.6; no longer J39.6
- net INTFC_NC4: now also J35.8; no longer J39.8
- net INTFC_NC7: now also J51.6; no longer J57.6
- net INTFC_NC8: now also J51.8; no longer J57.8
- net INTFC_SWDCLK1: now also J13.4; no longer J16.4
- net INTFC_SWDCLK2: now also J35.4; no longer J39.4
- net INTFC_SWDCLK3: now also J51.4; no longer J57.4
- net INTFC_SWDIO1: now also J13.2; no longer J16.2
- net INTFC_SWDIO2: now also J35.2; no longer J39.2
- net INTFC_SWDIO3: now also J51.2; no longer J57.2
- net N$11: now also J10.B5; no longer J13.B5
- net N$17: now also J10.A5; no longer J13.A5
- net N$33: now also J33.B5; no longer J37.B5
- net N$34: now also J33.A5; no longer J37.A5
- net N$49: now also J49.B5; no longer J55.B5
- net N$50: now also J49.A5; no longer J55.A5
- net SCL1: now also J15.4, J16.21; no longer J17.4, J18.21
- net SCL2: now also J36.4, J37.21; no longer J40.4, J41.21
- net SCL3: now also J52.4, J53.21; no longer J58.4, J59.21
- net SDA1: now also J15.3, J16.22; no longer J17.3, J18.22
- net SDA2: now also J36.3, J37.22; no longer J40.3, J41.22
- net SDA3: now also J52.3, J53.22; no longer J58.3, J59.22
- net TGT_SWCLK1: now also J11.4; no longer J15.4
- net TGT_SWCLK2: now also J34.4; no longer J38.4
- net TGT_SWCLK3: now also J50.4; no longer J56.4
- net TGT_SWDIO1: now also J11.2; no longer J15.2
- net TGT_SWDIO2: now also J34.2; no longer J38.2
- net TGT_SWDIO3: now also J50.2; no longer J56.2
- net TGT_SWO1: now also J11.6; no longer J15.6
- net TGT_SWO2: now also J34.6; no longer J38.6
- net TGT_SWO3: now also J50.6; no longer J56.6
- net USB_D+_R1: now also J10.A6, J10.B6; no longer J13.A6, J13.B6
- net USB_D+_R2: now also J33.A6, J33.B6; no longer J37.A6, J37.B6
- net USB_D+_R3: now also J49.A6, J49.B6; no longer J55.A6, J55.B6
- net USB_D-_R1: now also J10.A7, J10.B7; no longer J13.A7, J13.B7
- net USB_D-_R2: now also J33.A7, J33.B7; no longer J37.A7, J37.B7
- net USB_D-_R3: now also J49.A7, J49.B7; no longer J55.A7, J55.B7
- net V_USB1: now also J10.VBUS1, J10.VBUS2, J17.3, J17.3@2, J17.4, J17.4@2, J18.3, J18.4; no longer J13.VBUS1, J13.VBUS2, J19.3@2, J19.4@2, J20.3, J20.4, J21.3, J21.4
- net V_USB2: now also J33.VBUS1, J33.VBUS2, J38.3, J38.3@2, J38.4, J38.4@2, J39.3, J39.4, J40.3, J40.4; no longer J37.VBUS1, J37.VBUS2, J42.3, J42.3@2, J42.4, J42.4@2, J43.3, J43.4, J44.3, J44.4
- net V_USB3: now also J49.VBUS1, J49.VBUS2, J54.3, J54.3@2, J54.4, J54.4@2, J55.3, J55.4, J56.3, J56.4; no longer J55.VBUS1, J55.VBUS2, J60.3, J60.3@2, J60.4, J60.4@2, J61.3, J61.4, J62.3, J62.4
Other:
- board size 116.6 x 181.4 mm -> 119.1 x 178.8 mm
